Commit message: Adding bota force sensor w/ adaptater piece

File: xacro/gen3_w_bota_FT_sensor.in.xacro (robot description, xacro)
@@ -1,19 +1,49 @@
 <?xml version="1.0"?>
 <robot name="gen3" xmlns:xacro="http://ros.org/wiki/">
-    <!-- Arguments -->
-    <xacro:arg name="arm" default="gen3" />
-    <xacro:arg name="dof" default="7" />
-    <xacro:arg name="vision" default="true" />
-    <xacro:arg name="gripper" default="" />
-    <xacro:arg name="sim" default="false" />
-    <xacro:arg name="prefix" default="" />
-    <xacro:include filename="$(find kortex_description)/robots/kortex_robot.xacro" />
-    <xacro:load_robot arm="$(arg arm)" gripper="$(arg gripper)" dof="$(arg dof)" vision="$(arg vision)" sim="$(arg sim)" prefix="$(arg prefix)" />
-    <xacro:include filename="$(find rokubimini_description)/urdf/BFT_SENS_ECAT_M8.urdf.xacro" />
-    <xacro:BFT_SENS_ECAT_M8 prefix="FT_sensor" />
-    <joint name="robot_to_FT" type="fixed">
-      <parent link="end_effector_link" />
-      <child link="FT_sensor_mounting" />
-      <origin xyz="0.0 0.0 0.0" rpy="0.0 0.0 0.0" />
-    </joint>
+  <!-- Arguments -->
+  <xacro:arg name="arm" default="gen3" />
+  <xacro:arg name="dof" default="7" />
+  <xacro:arg name="vision" default="true" />
+  <xacro:arg name="gripper" default="" />
+  <xacro:arg name="sim" default="false" />
+  <xacro:arg name="prefix" default="" />
+  <xacro:arg name="meshPath" default="" />
+  <xacro:include filename="$(find kortex_description)/robots/kortex_robot.xacro" />
+  <xacro:load_robot arm="$(arg arm)" gripper="$(arg gripper)" dof="$(arg dof)"
+    vision="$(arg vision)" sim="$(arg sim)" prefix="$(arg prefix)" />
+  <xacro:include filename="$(find rokubimini_description)/urdf/BFT_SENS_ECAT_M8.urdf.xacro" />
+  <xacro:BFT_SENS_ECAT_M8 prefix="FT_sensor" />
+  <link name="FT_adapter">
+    <inertial>
+      <origin xyz="0.001329828523918 0.000509434161397 0.017297595549827" rpy="0 0 0" />
+      <mass value="0.12" />
+      <inertia ixx="5.40350E-05" ixy="8.13203E-08" ixz="1.70226E-06" iyy="5.69809E-05"
+        iyz="1.05961E-06" izz="8.81951E-05" />
+    </inertial>
+    <visual name="adapter">
+      <origin xyz="0 0 0" rpy="0 0 0" />
+      <geometry>
+        <mesh filename="$(arg meshPath)/force_sensor/adapter.STL" size="0.001 0.001 0.001" />
+      </geometry>
+      <material name="">
+        <color rgba="0.6902 0.61176 0.52941 1" />
+      </material>
+    </visual>
+    <collision>
+      <origin xyz="0 0 0.015" rpy="0 0 0" />
+      <geometry>
+        <cylinder radius="0.0075" length="0.03" />
+      </geometry>
+    </collision>
+  </link>
+  <joint name="kinova_to_adapter" type="fixed">
+    <parent link="end_effector_link" />
+    <child link="FT_adapter" />
+    <origin xyz="0.0 0.0 0.0" rpy="0.0 0.0 0.0" />
+  </joint>
+  <joint name="adapter_to_FT" type="fixed">
+    <parent link="FT_adapter" />
+    <child link="FT_sensor_mounting" />
+    <origin xyz="0.0 0.0 0.0" rpy="0.0 0.0 0.0" />
+  </joint>
 </robot>

Commit message: Fix bota force sensor implementation

File: xacro/gen3_w_bota_FT_sensor.in.xacro (robot description, xacro)
@@ -8,5 +8,4 @@
   <xacro:arg name="sim" default="false" />
   <xacro:arg name="prefix" default="" />
-  <xacro:arg name="meshPath" default="" />
   <xacro:include filename="$(find kortex_description)/robots/kortex_robot.xacro" />
   <xacro:load_robot arm="$(arg arm)" gripper="$(arg gripper)" dof="$(arg dof)"
@@ -22,7 +21,8 @@
     </inertial>
     <visual name="adapter">
-      <origin xyz="0 0 0" rpy="0 0 0" />
+      <origin xyz="0 0 0.0" rpy="0 0 0" />
       <geometry>
-        <mesh filename="$(arg meshPath)/force_sensor/adapter.STL" size="0.001 0.001 0.001" />
+        <mesh filename="file://@CMAKE_SOURCE_DIR@/meshes/force_sensor/adapter.STL"
+          scale="0.001 0.001 0.001" />
       </geometry>
       <material name="">
@@ -40,5 +40,5 @@
     <parent link="end_effector_link" />
     <child link="FT_adapter" />
-    <origin xyz="0.0 0.0 0.0" rpy="0.0 0.0 0.0" />
+    <origin xyz="0.0 0.0 0.03" rpy="0.0 0.0 0.0" />
   </joint>
   <joint name="adapter_to_FT" type="fixed">

Commit message: Add two variants to kinova's robot module and add a box for the DS4 at the end effector

File: xacro/gen3_w_bota_FT_sensor.in.xacro (robot description, xacro)
@@ -37,4 +37,27 @@
     </collision>
   </link>
+  <link name="DS4">
+    <inertial>
+      <origin xyz="0.0 0.0 0.04" rpy="0 0 0" />
+      <mass value="0.35" />
+      <inertia ixx="5.40350E-05" ixy="8.13203E-08" ixz="1.70226E-06" iyy="5.69809E-05"
+        iyz="1.05961E-06" izz="8.81951E-05" />
+    </inertial>
+    <visual name="ds4">
+      <origin xyz="0.01 0.01 0.025" rpy="0 0 0" />
+      <geometry>
+        <box size="0.02 0.02 0.2" />
+      </geometry>
+      <material name="">
+        <color rgba="0.6902 0.61176 0.52941 1" />
+      </material>
+    </visual>
+    <collision>
+      <origin xyz="0 0 0.015" rpy="0 0 0" />
+      <geometry>
+        <cylinder radius="0.0075" length="0.03" />
+      </geometry>
+    </collision>
+  </link>
   <joint name="kinova_to_adapter" type="fixed">
     <parent link="end_effector_link" />
@@ -47,3 +70,8 @@
     <origin xyz="0.0 0.0 0.0" rpy="0.0 0.0 0.0" />
   </joint>
+  <joint name="DS4_to_FT" type="fixed">
+    <parent link="FT_sensor_wrench" />
+    <child link="DS4" />
+    <origin xyz="0.0 0.0 0.0" rpy="0.0 0.0 0.0" />
+  </joint>
 </robot>

Commit message: Add DS4 controller equivalent body to robot model and rsdf file for potential contact surface

File: xacro/gen3_w_bota_FT_sensor.in.xacro (robot description, xacro)
@@ -45,7 +45,7 @@
     </inertial>
     <visual name="ds4">
-      <origin xyz="0.01 0.01 0.025" rpy="0 0 0" />
+      <origin xyz="0.0 0.0 0.03" rpy="0 0 0" />
       <geometry>
-        <box size="0.02 0.02 0.2" />
+        <box size="0.02 0.02 0.03" />
       </geometry>
       <material name="">
@@ -60,4 +60,5 @@
     </collision>
   </link>
+  <link name="DS4_tool"></link>
   <joint name="kinova_to_adapter" type="fixed">
     <parent link="end_effector_link" />
@@ -75,3 +76,8 @@
     <origin xyz="0.0 0.0 0.0" rpy="0.0 0.0 0.0" />
   </joint>
+  <joint name="DS4_to_tool" type="fixed">
+    <parent link="DS4" />
+    <child link="DS4_tool" />
+    <origin xyz="0.0 0.0 0.06" rpy="0.0 0.0 0.0" />
+  </joint>
 </robot>

Commit message: Updated rotor inertia and included DS4 holder model

File: xacro/gen3_w_bota_FT_sensor.in.xacro (robot description, xacro)
@@ -37,15 +37,15 @@
     </collision>
   </link>
-  <link name="DS4">
+  <link name="DS4_adapter">
     <inertial>
-      <origin xyz="0.0 0.0 0.04" rpy="0 0 0" />
-      <mass value="0.35" />
+      <origin xyz="-0.0001681638469675113 -0.0024779164507503317 0.059811455964133025" rpy="0 0 0" />
+      <mass value="0.0698" />
       <inertia ixx="5.40350E-05" ixy="8.13203E-08" ixz="1.70226E-06" iyy="5.69809E-05"
         iyz="1.05961E-06" izz="8.81951E-05" />
     </inertial>
-    <visual name="ds4">
-      <origin xyz="0.0 0.0 0.03" rpy="0 0 0" />
+    <visual name="ds4_adapter">
+      <origin xyz="0.0 0.0 0.0" rpy="0 0 0" />
       <geometry>
-        <box size="0.02 0.02 0.03" />
+        <mesh filename="file://@CMAKE_SOURCE_DIR@/meshes/DS4_adapter.STL" scale="0.001 0.001 0.001" />
       </geometry>
       <material name="">
@@ -57,4 +57,27 @@
       <geometry>
         <cylinder radius="0.0075" length="0.03" />
+      </geometry>
+    </collision>
+  </link>
+  <link name="DS4">
+    <inertial>
+      <origin xyz="0.0 0.0 0.045" rpy="0 0 0" />
+      <mass value="0.2162" />
+      <inertia ixx="5.40350E-05" ixy="8.13203E-08" ixz="1.70226E-06" iyy="5.69809E-05"
+        iyz="1.05961E-06" izz="8.81951E-05" />
+    </inertial>
+    <visual name="ds4">
+      <origin xyz="0.0 0.0 0.0" rpy="0 0 0" />
+      <geometry>
+        <box size="0.14 0.03 0.06" />
+      </geometry>
+      <material name="">
+        <color rgba="0.6902 0.61176 0.52941 1" />
+      </material>
+    </visual>
+    <collision>
+      <origin xyz="0 0 0.03" rpy="0 1.57 0" />
+      <geometry>
+        <cylinder radius="0.0075" length="0.14" />
       </geometry>
     </collision>
@@ -71,13 +94,18 @@
     <origin xyz="0.0 0.0 0.0" rpy="0.0 0.0 0.0" />
   </joint>
-  <joint name="DS4_to_FT" type="fixed">
+  <joint name="FT_to_DS4_adapter" type="fixed">
     <parent link="FT_sensor_wrench" />
+    <child link="DS4_adapter" />
+    <origin xyz="0.0 0.0 0.0" rpy="0.0 0.0 0.0" />
+  </joint>
+  <joint name="DS4_adapter_to_DS4" type="fixed">
+    <parent link="DS4_adapter" />
     <child link="DS4" />
-    <origin xyz="0.0 0.0 0.0" rpy="0.0 0.0 0.0" />
+    <origin xyz="0.0 0.0 0.08" rpy="0.0 0.0 0.0" />
   </joint>
   <joint name="DS4_to_tool" type="fixed">
     <parent link="DS4" />
     <child link="DS4_tool" />
-    <origin xyz="0.0 0.0 0.06" rpy="0.0 0.0 0.0" />
+    <origin xyz="0.0 0.0 0.0" rpy="0.0 0.0 0.0" />
   </joint>
 </robot>

Commit message: Add a bota only variant, updates to the handling of variants

File: xacro/gen3_w_bota_FT_sensor.in.xacro (robot description, xacro)
@@ -8,4 +8,5 @@
   <xacro:arg name="sim" default="false" />
   <xacro:arg name="prefix" default="" />
+  <xacro:arg name="DS4" default="false" />
   <xacro:include filename="$(find kortex_description)/robots/kortex_robot.xacro" />
   <xacro:load_robot arm="$(arg arm)" gripper="$(arg gripper)" dof="$(arg dof)"
@@ -37,51 +38,54 @@
     </collision>
   </link>
-  <link name="DS4_adapter">
-    <inertial>
-      <origin xyz="-0.0001681638469675113 -0.0024779164507503317 0.059811455964133025" rpy="0 0 0" />
-      <mass value="0.0698" />
-      <inertia ixx="5.40350E-05" ixy="8.13203E-08" ixz="1.70226E-06" iyy="5.69809E-05"
-        iyz="1.05961E-06" izz="8.81951E-05" />
-    </inertial>
-    <visual name="ds4_adapter">
-      <origin xyz="0.0 0.0 0.0" rpy="0 0 0" />
-      <geometry>
-        <mesh filename="file://@CMAKE_SOURCE_DIR@/meshes/DS4_adapter.STL" scale="0.001 0.001 0.001" />
-      </geometry>
-      <material name="">
-        <color rgba="0.6902 0.61176 0.52941 1" />
-      </material>
-    </visual>
-    <collision>
-      <origin xyz="0 0 0.015" rpy="0 0 0" />
-      <geometry>
-        <cylinder radius="0.0075" length="0.03" />
-      </geometry>
-    </collision>
-  </link>
-  <link name="DS4">
-    <inertial>
-      <origin xyz="0.0 0.0 0.045" rpy="0 0 0" />
-      <mass value="0.2162" />
-      <inertia ixx="5.40350E-05" ixy="8.13203E-08" ixz="1.70226E-06" iyy="5.69809E-05"
-        iyz="1.05961E-06" izz="8.81951E-05" />
-    </inertial>
-    <visual name="ds4">
-      <origin xyz="0.0 0.0 0.0" rpy="0 0 0" />
-      <geometry>
-        <box size="0.14 0.03 0.06" />
-      </geometry>
-      <material name="">
-        <color rgba="0.6902 0.61176 0.52941 1" />
-      </material>
-    </visual>
-    <collision>
-      <origin xyz="0 0 0.03" rpy="0 1.57 0" />
-      <geometry>
-        <cylinder radius="0.0075" length="0.14" />
-      </geometry>
-    </collision>
-  </link>
-  <link name="DS4_tool"></link>
+  <xacro:if value="$(arg DS4)">
+    <link name="DS4_adapter">
+      <inertial>
+        <origin xyz="-0.0001681638469675113 -0.0024779164507503317 0.059811455964133025" rpy="0 0 0" />
+        <mass value="0.0698" />
+        <inertia ixx="5.40350E-05" ixy="8.13203E-08" ixz="1.70226E-06" iyy="5.69809E-05"
+          iyz="1.05961E-06" izz="8.81951E-05" />
+      </inertial>
+      <visual name="ds4_adapter">
+        <origin xyz="0.0 0.0 0.0" rpy="0 0 0" />
+        <geometry>
+          <mesh filename="file://@CMAKE_SOURCE_DIR@/meshes/DS4_adapter.STL"
+            scale="0.001 0.001 0.001" />
+        </geometry>
+        <material name="">
+          <color rgba="0.6902 0.61176 0.52941 1" />
+        </material>
+      </visual>
+      <collision>
+        <origin xyz="0 0 0.015" rpy="0 0 0" />
+        <geometry>
+          <cylinder radius="0.0075" length="0.03" />
+        </geometry>
+      </collision>
+    </link>
+    <link name="DS4">
+      <inertial>
+        <origin xyz="0.0 0.0 0.045" rpy="0 0 0" />
+        <mass value="0.2162" />
+        <inertia ixx="5.40350E-05" ixy="8.13203E-08" ixz="1.70226E-06" iyy="5.69809E-05"
+          iyz="1.05961E-06" izz="8.81951E-05" />
+      </inertial>
+      <visual name="ds4">
+        <origin xyz="0.0 0.0 0.0" rpy="0 0 0" />
+        <geometry>
+          <box size="0.14 0.03 0.06" />
+        </geometry>
+        <material name="">
+          <color rgba="0.6902 0.61176 0.52941 1" />
+        </material>
+      </visual>
+      <collision>
+        <origin xyz="0 0 0.03" rpy="0 1.57 0" />
+        <geometry>
+          <cylinder radius="0.0075" length="0.14" />
+        </geometry>
+      </collision>
+    </link>
+    <link name="DS4_tool"></link>
+  </xacro:if>
   <joint name="kinova_to_adapter" type="fixed">
     <parent link="end_effector_link" />
@@ -94,18 +98,20 @@
     <origin xyz="0.0 0.0 0.0" rpy="0.0 0.0 0.0" />
   </joint>
-  <joint name="FT_to_DS4_adapter" type="fixed">
-    <parent link="FT_sensor_wrench" />
-    <child link="DS4_adapter" />
-    <origin xyz="0.0 0.0 0.0" rpy="0.0 0.0 0.0" />
-  </joint>
-  <joint name="DS4_adapter_to_DS4" type="fixed">
-    <parent link="DS4_adapter" />
-    <child link="DS4" />
-    <origin xyz="0.0 0.0 0.08" rpy="0.0 0.0 0.0" />
-  </joint>
-  <joint name="DS4_to_tool" type="fixed">
-    <parent link="DS4" />
-    <child link="DS4_tool" />
-    <origin xyz="0.0 0.0 0.0" rpy="0.0 0.0 0.0" />
-  </joint>
+  <xacro:if value="$(arg DS4)">
+    <joint name="FT_to_DS4_adapter" type="fixed">
+      <parent link="FT_sensor_wrench" />
+      <child link="DS4_adapter" />
+      <origin xyz="0.0 0.0 0.0" rpy="0.0 0.0 0.0" />
+    </joint>
+    <joint name="DS4_adapter_to_DS4" type="fixed">
+      <parent link="DS4_adapter" />
+      <child link="DS4" />
+      <origin xyz="0.0 0.0 0.08" rpy="0.0 0.0 0.0" />
+    </joint>
+    <joint name="DS4_to_tool" type="fixed">
+      <parent link="DS4" />
+      <child link="DS4_tool" />
+      <origin xyz="0.0 0.0 0.0" rpy="0.0 0.0 0.0" />
+    </joint>
+  </xacro:if>
 </robot>

Commit message: Update for ROS2

File: xacro/gen3_w_bota_FT_sensor.in.xacro (robot description, xacro)
@@ -2,14 +2,65 @@
 <robot name="gen3" xmlns:xacro="http://ros.org/wiki/">
   <!-- Arguments -->
+  <xacro:arg name="name" default="gen3_arm" />
+  <xacro:arg name="prefix" default="" />
   <xacro:arg name="arm" default="gen3" />
   <xacro:arg name="dof" default="7" />
   <xacro:arg name="vision" default="true" />
+  <xacro:arg name="robot_ip" default="192.168.0.1" />
+  <xacro:arg name="username" default="admin" />
+  <xacro:arg name="password" default="admin" />
+  <xacro:arg name="port" default="10000" />
+  <xacro:arg name="port_realtime" default="10001" />
+  <xacro:arg name="session_inactivity_timeout_ms" default="60000" />
+  <xacro:arg name="connection_inactivity_timeout_ms" default="2000" />
   <xacro:arg name="gripper" default="" />
-  <xacro:arg name="sim" default="false" />
-  <xacro:arg name="prefix" default="" />
+  <xacro:arg name="gripper_joint_name" default="finger_joint" />
+  <xacro:arg name="gripper_max_velocity" default="100.0" />
+  <xacro:arg name="gripper_max_force" default="100.0" />
+  <xacro:arg name="use_internal_bus_gripper_comm" default="false" />
+  <xacro:arg name="use_fake_hardware" default="false" />
+  <xacro:arg name="fake_sensor_commands" default="false" />
+  <xacro:arg name="sim_gazebo" default="false" />
+  <xacro:arg name="sim_isaac" default="false" />
+  <xacro:arg name="simulation_controllers"
+    default="$(find kortex_description)/arm/$(arg arm)/$(arg dof)dof/config/ros2_controllers.yaml" />
   <xacro:arg name="DS4" default="false" />
+  <!-- import main macro -->
   <xacro:include filename="$(find kortex_description)/robots/kortex_robot.xacro" />
-  <xacro:load_robot arm="$(arg arm)" gripper="$(arg gripper)" dof="$(arg dof)"
-    vision="$(arg vision)" sim="$(arg sim)" prefix="$(arg prefix)" />
+  <!-- convert to property to use substitution in function -->
+  <xacro:property name="initial_positions_file" default="$(arg initial_positions_file)" />
+  <!-- create link fixed to the "world" -->
+  <link name="world" />
+  <xacro:load_robot
+    parent="world"
+    arm="$(arg arm)"
+    gripper="$(arg gripper)"
+    gripper_joint_name="$(arg gripper_joint_name)"
+    gripper_max_velocity="$(arg gripper_max_velocity)"
+    gripper_max_force="$(arg gripper_max_force)"
+    dof="$(arg dof)"
+    vision="$(arg vision)"
+    robot_ip="$(arg robot_ip)"
+    username="$(arg username)"
+    password="$(arg password)"
+    port="$(arg port)"
+    port_realtime="$(arg port_realtime)"
+    session_inactivity_timeout_ms="$(arg session_inactivity_timeout_ms)"
+    connection_inactivity_timeout_ms="$(arg connection_inactivity_timeout_ms)"
+    use_internal_bus_gripper_comm="$(arg use_internal_bus_gripper_comm)"
+    prefix="$(arg prefix)"
+    use_fake_hardware="$(arg use_fake_hardware)"
+    fake_sensor_commands="$(arg fake_sensor_commands)"
+    sim_gazebo="$(arg sim_gazebo)"
+    sim_isaac="$(arg sim_isaac)">
+    <origin xyz="0 0 0" rpy="0 0 0" />
+  </xacro:load_robot>
+  <xacro:if value="$(arg sim_gazebo)">
+    <gazebo reference="world">
+      <plugin filename="libgazebo_ros2_control.so" name="gazebo_ros2_control">
+        <parameters>$(arg simulation_controllers)</parameters>
+      </plugin>
+    </gazebo>
+  </xacro:if>
   <xacro:include filename="$(find rokubimini_description)/urdf/BFT_SENS_ECAT_M8.urdf.xacro" />
   <xacro:BFT_SENS_ECAT_M8 prefix="FT_sensor" />
