Commit message: add default kinova

File: xacro/gen3_w_bota_FT_sensor.in.xacro (robot description, xacro)
@@ -26,4 +26,5 @@
     default="$(find kortex_description)/arm/$(arg arm)/$(arg dof)dof/config/ros2_controllers.yaml" />
   <xacro:arg name="DS4" default="false" />
+  <xacro:arg name="bota" default="true" />
   <!-- import main macro -->
   <xacro:include filename="$(find kortex_description)/robots/kortex_robot.xacro" />
@@ -63,42 +64,18 @@
     </gazebo>
   </xacro:if>
-  <xacro:include filename="$(find rokubimini_description)/urdf/BFT_SENS_ECAT_M8.urdf.xacro" />
-  <xacro:BFT_SENS_ECAT_M8 prefix="FT_sensor" />
-  <link name="FT_adapter">
-    <inertial>
-      <origin xyz="0.001329828523918 0.000509434161397 0.017297595549827" rpy="0 0 0" />
-      <mass value="0.12" />
-      <inertia ixx="5.40350E-05" ixy="8.13203E-08" ixz="1.70226E-06" iyy="5.69809E-05"
-        iyz="1.05961E-06" izz="8.81951E-05" />
-    </inertial>
-    <visual name="adapter">
-      <origin xyz="0 0 0.0" rpy="0 0 0" />
-      <geometry>
-        <mesh filename="file://@CMAKE_SOURCE_DIR@/meshes/force_sensor/adapter.STL"
-          scale="0.001 0.001 0.001" />
-      </geometry>
-      <material name="">
-        <color rgba="0.6902 0.61176 0.52941 1" />
-      </material>
-    </visual>
-    <collision>
-      <origin xyz="0 0 0.015" rpy="0 0 0" />
-      <geometry>
-        <cylinder radius="0.0075" length="0.03" />
-      </geometry>
-    </collision>
-  </link>
-  <xacro:if value="$(arg DS4)">
-    <link name="DS4_adapter">
+  <xacro:if value="$(arg bota)">
+    <xacro:include filename="$(find rokubimini_description)/urdf/BFT_SENS_ECAT_M8.urdf.xacro" />
+    <xacro:BFT_SENS_ECAT_M8 prefix="FT_sensor" />
+    <link name="FT_adapter">
       <inertial>
-        <origin xyz="-0.0001681638469675113 -0.0024779164507503317 0.059811455964133025" rpy="0 0 0" />
-        <mass value="0.0698" />
+        <origin xyz="0.001329828523918 0.000509434161397 0.017297595549827" rpy="0 0 0" />
+        <mass value="0.12" />
         <inertia ixx="5.40350E-05" ixy="8.13203E-08" ixz="1.70226E-06" iyy="5.69809E-05"
           iyz="1.05961E-06" izz="8.81951E-05" />
       </inertial>
-      <visual name="ds4_adapter">
-        <origin xyz="0.0 0.0 0.0" rpy="0 0 0" />
+      <visual name="adapter">
+        <origin xyz="0 0 0.0" rpy="0 0 0" />
         <geometry>
-          <mesh filename="file://@CMAKE_SOURCE_DIR@/meshes/DS4_adapter.STL"
+          <mesh filename="file://@CMAKE_SOURCE_DIR@/meshes/force_sensor/adapter.STL"
             scale="0.001 0.001 0.001" />
         </geometry>
@@ -114,55 +91,81 @@
       </collision>
     </link>
-    <link name="DS4">
-      <inertial>
-        <origin xyz="0.0 0.0 0.045" rpy="0 0 0" />
-        <mass value="0.2162" />
-        <inertia ixx="5.40350E-05" ixy="8.13203E-08" ixz="1.70226E-06" iyy="5.69809E-05"
-          iyz="1.05961E-06" izz="8.81951E-05" />
-      </inertial>
-      <visual name="ds4">
-        <origin xyz="0.0 0.0 0.0" rpy="0 0 0" />
-        <geometry>
-          <box size="0.14 0.03 0.06" />
-        </geometry>
-        <material name="">
-          <color rgba="0.6902 0.61176 0.52941 1" />
-        </material>
-      </visual>
-      <collision>
-        <origin xyz="0 0 0.03" rpy="0 1.57 0" />
-        <geometry>
-          <cylinder radius="0.0075" length="0.14" />
-        </geometry>
-      </collision>
-    </link>
-    <link name="DS4_tool"></link>
-  </xacro:if>
-  <joint name="kinova_to_adapter" type="fixed">
-    <parent link="end_effector_link" />
-    <child link="FT_adapter" />
-    <origin xyz="0.0 0.0 0.03" rpy="0.0 0.0 0.0" />
-  </joint>
-  <joint name="adapter_to_FT" type="fixed">
-    <parent link="FT_adapter" />
-    <child link="FT_sensor_mounting" />
-    <origin xyz="0.0 0.0 0.0" rpy="0.0 0.0 0.0" />
-  </joint>
-  <xacro:if value="$(arg DS4)">
-    <joint name="FT_to_DS4_adapter" type="fixed">
-      <parent link="FT_sensor_wrench" />
-      <child link="DS4_adapter" />
+    <xacro:if value="$(arg DS4)">
+      <link name="DS4_adapter">
+        <inertial>
+          <origin xyz="-0.0001681638469675113 -0.0024779164507503317 0.059811455964133025" rpy="0 0 0" />
+          <mass value="0.0698" />
+          <inertia ixx="5.40350E-05" ixy="8.13203E-08" ixz="1.70226E-06" iyy="5.69809E-05"
+            iyz="1.05961E-06" izz="8.81951E-05" />
+        </inertial>
+        <visual name="ds4_adapter">
+          <origin xyz="0.0 0.0 0.0" rpy="0 0 0" />
+          <geometry>
+            <mesh filename="file://@CMAKE_SOURCE_DIR@/meshes/DS4_adapter.STL"
+              scale="0.001 0.001 0.001" />
+          </geometry>
+          <material name="">
+            <color rgba="0.6902 0.61176 0.52941 1" />
+          </material>
+        </visual>
+        <collision>
+          <origin xyz="0 0 0.015" rpy="0 0 0" />
+          <geometry>
+            <cylinder radius="0.0075" length="0.03" />
+          </geometry>
+        </collision>
+      </link>
+      <link name="DS4">
+        <inertial>
+          <origin xyz="0.0 0.0 0.045" rpy="0 0 0" />
+          <mass value="0.2162" />
+          <inertia ixx="5.40350E-05" ixy="8.13203E-08" ixz="1.70226E-06" iyy="5.69809E-05"
+            iyz="1.05961E-06" izz="8.81951E-05" />
+        </inertial>
+        <visual name="ds4">
+          <origin xyz="0.0 0.0 0.0" rpy="0 0 0" />
+          <geometry>
+            <box size="0.14 0.03 0.06" />
+          </geometry>
+          <material name="">
+            <color rgba="0.6902 0.61176 0.52941 1" />
+          </material>
+        </visual>
+        <collision>
+          <origin xyz="0 0 0.03" rpy="0 1.57 0" />
+          <geometry>
+            <cylinder radius="0.0075" length="0.14" />
+          </geometry>
+        </collision>
+      </link>
+      <link name="DS4_tool"></link>
+    </xacro:if>
+    <joint name="kinova_to_adapter" type="fixed">
+      <parent link="end_effector_link" />
+      <child link="FT_adapter" />
+      <origin xyz="0.0 0.0 0.03" rpy="0.0 0.0 0.0" />
+    </joint>
+    <joint name="adapter_to_FT" type="fixed">
+      <parent link="FT_adapter" />
+      <child link="FT_sensor_mounting" />
       <origin xyz="0.0 0.0 0.0" rpy="0.0 0.0 0.0" />
     </joint>
-    <joint name="DS4_adapter_to_DS4" type="fixed">
-      <parent link="DS4_adapter" />
-      <child link="DS4" />
-      <origin xyz="0.0 0.0 0.08" rpy="0.0 0.0 0.0" />
-    </joint>
-    <joint name="DS4_to_tool" type="fixed">
-      <parent link="DS4" />
-      <child link="DS4_tool" />
-      <origin xyz="0.0 0.0 0.0" rpy="0.0 0.0 0.0" />
-    </joint>
+    <xacro:if value="$(arg DS4)">
+      <joint name="FT_to_DS4_adapter" type="fixed">
+        <parent link="FT_sensor_wrench" />
+        <child link="DS4_adapter" />
+        <origin xyz="0.0 0.0 0.0" rpy="0.0 0.0 0.0" />
+      </joint>
+      <joint name="DS4_adapter_to_DS4" type="fixed">
+        <parent link="DS4_adapter" />
+        <child link="DS4" />
+        <origin xyz="0.0 0.0 0.08" rpy="0.0 0.0 0.0" />
+      </joint>
+      <joint name="DS4_to_tool" type="fixed">
+        <parent link="DS4" />
+        <child link="DS4_tool" />
+        <origin xyz="0.0 0.0 0.0" rpy="0.0 0.0 0.0" />
+      </joint>
+    </xacro:if>
   </xacro:if>
-</robot>
+  </robot>

Commit message: add kinova camera version with and without gripper

File: xacro/gen3_w_bota_FT_sensor.in.xacro (robot description, xacro)
@@ -77,6 +77,5 @@
         <origin xyz="0 0 0.0" rpy="0 0 0" />
         <geometry>
-          <mesh filename="file://@CMAKE_SOURCE_DIR@/meshes/force_sensor/adapter.STL"
-            scale="0.001 0.001 0.001" />
+          <mesh filename="file://@CMAKE_SOURCE_DIR@/meshes/adapter.STL" />
         </geometry>
         <material name="">
@@ -102,6 +101,5 @@
           <origin xyz="0.0 0.0 0.0" rpy="0 0 0" />
           <geometry>
-            <mesh filename="file://@CMAKE_SOURCE_DIR@/meshes/DS4_adapter.STL"
-              scale="0.001 0.001 0.001" />
+            <mesh filename="file://@CMAKE_SOURCE_DIR@/meshes/DS4_adapter.STL" />
           </geometry>
           <material name="">
