Commit message: Refine GenA Bota sensor mounting

File: xacro/BFT_KG3_IND2_SW.urdf.xacro (robot description, xacro)
@@ -10,7 +10,7 @@
       </inertial>
       <visual>
-        <origin xyz="0 0 0" rpy="0 0 0" />
+        <origin xyz="0 0 0.014" rpy="0 0 0" />
         <geometry>
-          <mesh filename="package://mc_kinova/meshes/BFT_KG3_IND2_SW/mounting.dae" scale="0.001 0.001 0.001" />
+          <cylinder radius="0.035" length="0.028" />
         </geometry>
         <material name="">
@@ -19,5 +19,5 @@
       </visual>
       <collision>
-        <origin xyz="0 0 0" rpy="0 0 0" />
+        <origin xyz="0 0 0.014" rpy="0 0 0" />
         <geometry>
           <cylinder radius="0.035" length="0.028" />

File: xacro/gen3.in.xacro (robot description, xacro)
@@ -67,5 +67,5 @@
   <xacro:if value="$(arg bota)">
     <xacro:if value="$(eval bota_version == 'gena')">
-      <xacro:include filename="@CMAKE_SOURCE_DIR@/xacro/BFT_KG3_IND2_SW.urdf.xacro" />
+      <xacro:include filename="@KINOVA_BOTA_GENA_XACRO_PATH@" />
       <xacro:BFT_KG3_IND2_SW prefix="FT_sensor" />
     </xacro:if>
@@ -74,27 +74,29 @@
       <xacro:BFT_SENS_ECAT_M8 prefix="FT_sensor" />
     </xacro:unless>
-    <link name="FT_adapter">
-      <inertial>
-        <origin xyz="0.001329828523918 0.000509434161397 0.017297595549827" rpy="0 0 0" />
-        <mass value="0.12" />
-        <inertia ixx="5.40350E-05" ixy="8.13203E-08" ixz="1.70226E-06" iyy="5.69809E-05"
-          iyz="1.05961E-06" izz="8.81951E-05" />
-      </inertial>
-      <visual name="adapter">
-        <origin xyz="0 0 0.0" rpy="0 0 0" />
-        <geometry>
-          <mesh filename="file://@CMAKE_SOURCE_DIR@/meshes/adapter.STL" />
-        </geometry>
-        <material name="">
-          <color rgba="0.6902 0.61176 0.52941 1" />
-        </material>
-      </visual>
-      <collision>
-        <origin xyz="0 0 0.015" rpy="0 0 0" />
-        <geometry>
-          <cylinder radius="0.0075" length="0.03" />
-        </geometry>
-      </collision>
-    </link>
+    <xacro:unless value="$(eval bota_version == 'gena')">
+      <link name="FT_adapter">
+        <inertial>
+          <origin xyz="0.001329828523918 0.000509434161397 0.017297595549827" rpy="0 0 0" />
+          <mass value="0.12" />
+          <inertia ixx="5.40350E-05" ixy="8.13203E-08" ixz="1.70226E-06" iyy="5.69809E-05"
+            iyz="1.05961E-06" izz="8.81951E-05" />
+        </inertial>
+        <visual name="adapter">
+          <origin xyz="0 0 0.0" rpy="0 0 0" />
+          <geometry>
+            <mesh filename="file://@CMAKE_SOURCE_DIR@/meshes/adapter.STL" />
+          </geometry>
+          <material name="">
+            <color rgba="0.6902 0.61176 0.52941 1" />
+          </material>
+        </visual>
+        <collision>
+          <origin xyz="0 0 0.015" rpy="0 0 0" />
+          <geometry>
+            <cylinder radius="0.0075" length="0.03" />
+          </geometry>
+        </collision>
+      </link>
+    </xacro:unless>
     <xacro:if value="$(eval end_effector == 'ds4')">
       <link name="DS4_adapter">
@@ -146,14 +148,23 @@
       <link name="DS4_tool"></link>
     </xacro:if>
-    <joint name="kinova_to_adapter" type="fixed">
-      <parent link="end_effector_link" />
-      <child link="FT_adapter" />
-      <origin xyz="0.0 0.0 0.03" rpy="0.0 0.0 0.0" />
-    </joint>
-    <joint name="adapter_to_FT" type="fixed">
-      <parent link="FT_adapter" />
-      <child link="FT_sensor_mounting" />
-      <origin xyz="0.0 0.0 0.0" rpy="0.0 0.0 0.0" />
-    </joint>
+    <xacro:if value="$(eval bota_version == 'gena')">
+      <joint name="kinova_to_FT" type="fixed">
+        <parent link="end_effector_link" />
+        <child link="FT_sensor_mounting" />
+        <origin xyz="0.0 0.0 0.0" rpy="0.0 0.0 0.0" />
+      </joint>
+    </xacro:if>
+    <xacro:unless value="$(eval bota_version == 'gena')">
+      <joint name="kinova_to_adapter" type="fixed">
+        <parent link="end_effector_link" />
+        <child link="FT_adapter" />
+        <origin xyz="0.0 0.0 0.03" rpy="0.0 0.0 0.0" />
+      </joint>
+      <joint name="adapter_to_FT" type="fixed">
+        <parent link="FT_adapter" />
+        <child link="FT_sensor_mounting" />
+        <origin xyz="0.0 0.0 0.0" rpy="0.0 0.0 0.0" />
+      </joint>
+    </xacro:unless>
     <xacro:if value="$(eval end_effector == 'ds4')">
       <joint name="FT_to_DS4_adapter" type="fixed">

File: xacro/gen3_bota.in.xacro (robot description, xacro)
@@ -67,5 +67,5 @@
   <xacro:if value="$(arg bota)">
     <xacro:if value="$(eval bota_version == 'gena')">
-      <xacro:include filename="@CMAKE_SOURCE_DIR@/xacro/BFT_KG3_IND2_SW.urdf.xacro" />
+      <xacro:include filename="@KINOVA_BOTA_GENA_XACRO_PATH@" />
       <xacro:BFT_KG3_IND2_SW prefix="FT_sensor" />
     </xacro:if>
@@ -74,27 +74,29 @@
       <xacro:BFT_SENS_ECAT_M8 prefix="FT_sensor" />
     </xacro:unless>
-    <link name="FT_adapter">
-      <inertial>
-        <origin xyz="0.001329828523918 0.000509434161397 0.017297595549827" rpy="0 0 0" />
-        <mass value="0.12" />
-        <inertia ixx="5.40350E-05" ixy="8.13203E-08" ixz="1.70226E-06" iyy="5.69809E-05"
-          iyz="1.05961E-06" izz="8.81951E-05" />
-      </inertial>
-      <visual name="adapter">
-        <origin xyz="0 0 0.0" rpy="0 0 0" />
-        <geometry>
-          <mesh filename="file://@CMAKE_SOURCE_DIR@/meshes/adapter.STL" />
-        </geometry>
-        <material name="">
-          <color rgba="0.6902 0.61176 0.52941 1" />
-        </material>
-      </visual>
-      <collision>
-        <origin xyz="0 0 0.015" rpy="0 0 0" />
-        <geometry>
-          <cylinder radius="0.0075" length="0.03" />
-        </geometry>
-      </collision>
-    </link>
+    <xacro:unless value="$(eval bota_version == 'gena')">
+      <link name="FT_adapter">
+        <inertial>
+          <origin xyz="0.001329828523918 0.000509434161397 0.017297595549827" rpy="0 0 0" />
+          <mass value="0.12" />
+          <inertia ixx="5.40350E-05" ixy="8.13203E-08" ixz="1.70226E-06" iyy="5.69809E-05"
+            iyz="1.05961E-06" izz="8.81951E-05" />
+        </inertial>
+        <visual name="adapter">
+          <origin xyz="0 0 0.0" rpy="0 0 0" />
+          <geometry>
+            <mesh filename="file://@CMAKE_SOURCE_DIR@/meshes/adapter.STL" />
+          </geometry>
+          <material name="">
+            <color rgba="0.6902 0.61176 0.52941 1" />
+          </material>
+        </visual>
+        <collision>
+          <origin xyz="0 0 0.015" rpy="0 0 0" />
+          <geometry>
+            <cylinder radius="0.0075" length="0.03" />
+          </geometry>
+        </collision>
+      </link>
+    </xacro:unless>
     <xacro:if value="$(eval end_effector == 'none')">
       <link name="tool"></link>
@@ -201,14 +203,23 @@
       <link name="tool"></link>
     </xacro:if>
-    <joint name="kinova_to_adapter" type="fixed">
-      <parent link="end_effector_link" />
-      <child link="FT_adapter" />
-      <origin xyz="0.0 0.0 0.03" rpy="0.0 0.0 0.0" />
-    </joint>
-    <joint name="adapter_to_FT" type="fixed">
-      <parent link="FT_adapter" />
-      <child link="FT_sensor_mounting" />
-      <origin xyz="0.0 0.0 0.0" rpy="0.0 0.0 0.0" />
-    </joint>
+    <xacro:if value="$(eval bota_version == 'gena')">
+      <joint name="kinova_to_FT" type="fixed">
+        <parent link="end_effector_link" />
+        <child link="FT_sensor_mounting" />
+        <origin xyz="0.0 0.0 0.0" rpy="0.0 0.0 0.0" />
+      </joint>
+    </xacro:if>
+    <xacro:unless value="$(eval bota_version == 'gena')">
+      <joint name="kinova_to_adapter" type="fixed">
+        <parent link="end_effector_link" />
+        <child link="FT_adapter" />
+        <origin xyz="0.0 0.0 0.03" rpy="0.0 0.0 0.0" />
+      </joint>
+      <joint name="adapter_to_FT" type="fixed">
+        <parent link="FT_adapter" />
+        <child link="FT_sensor_mounting" />
+        <origin xyz="0.0 0.0 0.0" rpy="0.0 0.0 0.0" />
+      </joint>
+    </xacro:unless>
     <xacro:if value="$(eval end_effector == 'none')">
       <joint name="FT_to_tool" type="fixed">

Commit message: Use STL mesh for GenA sensor visual

File: xacro/BFT_KG3_IND2_SW.urdf.xacro (robot description, xacro)
@@ -10,7 +10,7 @@
       </inertial>
       <visual>
-        <origin xyz="0 0 0.014" rpy="0 0 0" />
+        <origin xyz="0 0 0" rpy="0 0 -1.57079632679" />
         <geometry>
-          <cylinder radius="0.035" length="0.028" />
+          <mesh filename="file://@CMAKE_SOURCE_DIR@/meshes/BFT_KG3_IND2_SW/mounting.stl" scale="0.001 0.001 0.001" />
         </geometry>
         <material name="">
@@ -19,5 +19,5 @@
       </visual>
       <collision>
-        <origin xyz="0 0 0.014" rpy="0 0 0" />
+        <origin xyz="0 0 0" rpy="0 0 0" />
         <geometry>
           <cylinder radius="0.035" length="0.028" />

Commit message: Fix GenA FT sensor frame in xacro

File: xacro/BFT_KG3_IND2_SW.urdf.xacro (robot description, xacro)
@@ -34,5 +34,5 @@
     </link>
     <joint name="${prefix}_mounting_to_imu" type="fixed">
-      <origin xyz="0.0197035899999985 0.00748612999999993 0.0077875000000011" rpy="0 0 0" />
+      <origin xyz="0.0197035899999985 0.00748612999999993 0.0077875000000011" rpy="0 0 1.57079632679" />
       <parent link="${prefix}_mounting" />
       <child link="${prefix}_imu" />
@@ -48,9 +48,16 @@
     </link>
     <joint name="${prefix}_mounting_to_wrench" type="fixed">
-      <origin xyz="0 0 0.0379800000000009" rpy="0 0 0" />
+      <origin xyz="0 0 0.0379800000000009" rpy="0 0 1.57079632679" />
       <parent link="${prefix}_mounting" />
       <child link="${prefix}_wrench" />
       <axis xyz="0 0 0" />
     </joint>
+    <link name="${prefix}_tool_frame"/>
+    <joint name="${prefix}_wrench_to_tool_frame" type="fixed">
+      <origin xyz="0 0 0" rpy="0 0 -1.57079632679" />
+      <parent link="${prefix}_wrench" />
+      <child link="${prefix}_tool_frame" />
+      <axis xyz="0 0 0" />
+    </joint>
   </xacro:macro>
 </robot>

File: xacro/gen3.in.xacro (robot description, xacro)
@@ -194,5 +194,5 @@
     <xacro:if value="$(eval end_effector == 'ds4')">
       <joint name="FT_to_DS4_adapter" type="fixed">
-        <parent link="FT_sensor_wrench" />
+        <parent link="FT_sensor_tool_frame" />
         <child link="DS4_adapter" />
         <origin xyz="0.0 0.0 0.0" rpy="0.0 0.0 0.0" />

File: xacro/gen3_bota.in.xacro (robot description, xacro)
@@ -229,5 +229,5 @@
     <xacro:if value="$(eval end_effector == 'none')">
       <joint name="FT_to_tool" type="fixed">
-        <parent link="FT_sensor_wrench" />
+        <parent link="FT_sensor_tool_frame" />
         <child link="tool" />
         <origin xyz="0.0 0.0 0.0" rpy="0.0 0.0 0.0" />
@@ -236,5 +236,5 @@
     <xacro:if value="$(eval end_effector == 'ds4')">
       <joint name="FT_to_DS4_adapter" type="fixed">
-        <parent link="FT_sensor_wrench" />
+        <parent link="FT_sensor_tool_frame" />
         <child link="DS4_adapter" />
         <origin xyz="0.0 0.0 0.0" rpy="0.0 0.0 0.0" />
@@ -253,5 +253,5 @@
     <xacro:if value="$(eval end_effector == 'plate')">
       <joint name="FT_to_plate" type="fixed">
-        <parent link="FT_sensor_wrench" />
+        <parent link="FT_sensor_tool_frame" />
         <child link="plate" />
         <origin xyz="0.0 0.0 0.0" rpy="0.0 0.0 0.0" />
@@ -265,5 +265,5 @@
     <xacro:if value="$(eval end_effector == 'screw')">
       <joint name="FT_to_screw" type="fixed">
-        <parent link="FT_sensor_wrench" />
+        <parent link="FT_sensor_tool_frame" />
         <child link="screw" />
         <origin xyz="0.0 0.0 0.0" rpy="0.0 0.0 0.0" />

Commit message: Flip GenA FT sensor frame rotation

File: xacro/BFT_KG3_IND2_SW.urdf.xacro (robot description, xacro)
@@ -34,5 +34,5 @@
     </link>
     <joint name="${prefix}_mounting_to_imu" type="fixed">
-      <origin xyz="0.0197035899999985 0.00748612999999993 0.0077875000000011" rpy="0 0 1.57079632679" />
+      <origin xyz="0.0197035899999985 0.00748612999999993 0.0077875000000011" rpy="0 0 -1.57079632679" />
       <parent link="${prefix}_mounting" />
       <child link="${prefix}_imu" />
@@ -48,5 +48,5 @@
     </link>
     <joint name="${prefix}_mounting_to_wrench" type="fixed">
-      <origin xyz="0 0 0.0379800000000009" rpy="0 0 1.57079632679" />
+      <origin xyz="0 0 0.0379800000000009" rpy="0 0 -1.57079632679" />
       <parent link="${prefix}_mounting" />
       <child link="${prefix}_wrench" />
@@ -55,5 +55,5 @@
     <link name="${prefix}_tool_frame"/>
     <joint name="${prefix}_wrench_to_tool_frame" type="fixed">
-      <origin xyz="0 0 0" rpy="0 0 -1.57079632679" />
+      <origin xyz="0 0 0" rpy="0 0 1.57079632679" />
       <parent link="${prefix}_wrench" />
       <child link="${prefix}_tool_frame" />
