Commit message: Add KinovaBotaPlate variant

File: xacro/gen3_bota.in.xacro (robot description, xacro)
@@ -26,4 +26,5 @@
     default="$(find kortex_description)/arm/$(arg arm)/$(arg dof)dof/config/ros2_controllers.yaml" />
   <xacro:arg name="DS4" default="false" />
+  <xacro:arg name="plate" default="false" />
   <xacro:arg name="bota" default="true" />
   <!-- import main macro -->
@@ -139,4 +140,30 @@
       <link name="DS4_tool"></link>
     </xacro:if>
+    <xacro:if value="$(arg plate)">
+      <link name="plate">
+        <inertial>
+          <origin xyz="-0.0001681638469675113 -0.0024779164507503317 0.059811455964133025" rpy="0 0 0" />
+          <mass value="0.0698" />
+          <inertia ixx="5.40350E-05" ixy="8.13203E-08" ixz="1.70226E-06" iyy="5.69809E-05"
+            iyz="1.05961E-06" izz="8.81951E-05" />
+        </inertial>
+        <visual name="ds4_adapter">
+          <origin xyz="0.0 0.0 0.0" rpy="0 0 0" />
+          <geometry>
+            <mesh filename="file://@CMAKE_SOURCE_DIR@/meshes/plate.STL" />
+          </geometry>
+          <material name="">
+            <color rgba="0.6902 0.61176 0.52941 1" />
+          </material>
+        </visual>
+        <collision>
+          <origin xyz="0 0 0.015" rpy="0 0 0" />
+          <geometry>
+            <cylinder radius="0.0075" length="0.03" />
+          </geometry>
+        </collision>
+      </link>
+      <link name="plate_tool"></link>
+    </xacro:if>
     <joint name="kinova_to_adapter" type="fixed">
       <parent link="end_effector_link" />
@@ -166,4 +193,16 @@
       </joint>
     </xacro:if>
+    <xacro:if value="$(arg plate)">
+      <joint name="FT_to_plate" type="fixed">
+        <parent link="FT_sensor_wrench" />
+        <child link="plate" />
+        <origin xyz="0.0 0.0 0.0" rpy="0.0 0.0 0.0" />
+      </joint>
+      <joint name="plate_to_tool" type="fixed">
+        <parent link="plate" />
+        <child link="plate_tool" />
+        <origin xyz="0.0 0.0 0.0" rpy="0.0 0.0 0.0" />
+      </joint>
+    </xacro:if>
   </xacro:if>
   </robot>

Commit message: Fix Gen0 Bota tool frame URDF

File: xacro/gen3_bota.in.xacro (robot description, xacro)
@@ -78,4 +78,10 @@
       <xacro:include filename="$(find rokubimini_description)/urdf/BFT_SENS_ECAT_M8.urdf.xacro" />
       <xacro:BFT_SENS_ECAT_M8 prefix="FT_sensor" />
+      <link name="FT_sensor_tool_frame" />
+      <joint name="FT_sensor_wrench_to_tool_frame" type="fixed">
+        <parent link="FT_sensor_wrench" />
+        <child link="FT_sensor_tool_frame" />
+        <origin xyz="0 0 0" rpy="0 0 0" />
+      </joint>
     </xacro:unless>
     <xacro:unless value="$(eval bota_version == 'gena')">

Commit message: feat(new frame): Add racquet_frame frame to KinovaBotaPlate variant

File: xacro/gen3_bota.in.xacro (robot description, xacro)
@@ -286,4 +286,10 @@
         <origin xyz="0.0 0.0 0.0" rpy="0.0 0.0 0.0" />
       </joint>
+      <link name="racquet_frame"></link>
+      <joint name="plate_to_racquet_frame" type="fixed">
+        <parent link="plate" />
+        <child link="racquet_frame" />
+        <origin xyz="0.0 -0.125 0.0" rpy="0.0 0.78539816339 0.0" />
+      </joint>
       <joint name="plate_to_tool" type="fixed">
         <parent link="plate" />

Commit message: fix(racquet frame): Fix issue with new racquet frame conversion from XML

File: xacro/gen3_bota.in.xacro (robot description, xacro)
@@ -290,5 +290,5 @@
         <parent link="plate" />
         <child link="racquet_frame" />
-        <origin xyz="0.0 -0.125 0.0" rpy="0.0 0.78539816339 0.0" />
+        <origin xyz="0.0 0.0 0.125" rpy="-1.57079632679 0.0 0.0" />
       </joint>
       <joint name="plate_to_tool" type="fixed">
