Commit message: Fix raquet weight and Optional in CMakeLists

File: xacro/gen3_bota.in.xacro (robot description, xacro)
@@ -162,8 +162,8 @@
       <link name="plate">
         <inertial>
-          <origin xyz="-0.0001681638469675113 -0.0024779164507503317 0.059811455964133025" rpy="0 0 0" />
-          <mass value="0.0698" />
-          <inertia ixx="5.40350E-05" ixy="8.13203E-08" ixz="1.70226E-06" iyy="5.69809E-05"
-            iyz="1.05961E-06" izz="8.81951E-05" />
+          <origin xyz="-1.58E-05 -9.40E-02 1.58E-05" rpy="0 0 0" />
+          <mass value="0.1" />
+          <inertia ixx="5.58925E-04" iyy="1.45301E-04" izz="5.58925E-04"
+                  ixy="1.52637E-07" ixz="6.50849E-05" iyz="-1.52637E-07" />
         </inertial>
         <visual name="plate">
@@ -290,5 +290,5 @@
         <parent link="plate" />
         <child link="racquet_frame" />
-        <origin xyz="0.0 0.0 0.125" rpy="-1.57079632679 0.0 0.0" />
+        <origin xyz="0.0 -0.125 0.0" rpy="0.0 0.78539816339 0.0" />
       </joint>
       <joint name="plate_to_tool" type="fixed">

Commit message: Revert "Fix raquet weight and Optional in CMakeLists"
This reverts commit 56be37f75515dd75eed03295f803ce7f3f27b2f1.

File: xacro/gen3_bota.in.xacro (robot description, xacro)
@@ -162,8 +162,8 @@
       <link name="plate">
         <inertial>
-          <origin xyz="-1.58E-05 -9.40E-02 1.58E-05" rpy="0 0 0" />
-          <mass value="0.1" />
-          <inertia ixx="5.58925E-04" iyy="1.45301E-04" izz="5.58925E-04"
-                  ixy="1.52637E-07" ixz="6.50849E-05" iyz="-1.52637E-07" />
+          <origin xyz="-0.0001681638469675113 -0.0024779164507503317 0.059811455964133025" rpy="0 0 0" />
+          <mass value="0.0698" />
+          <inertia ixx="5.40350E-05" ixy="8.13203E-08" ixz="1.70226E-06" iyy="5.69809E-05"
+            iyz="1.05961E-06" izz="8.81951E-05" />
         </inertial>
         <visual name="plate">
@@ -290,5 +290,5 @@
         <parent link="plate" />
         <child link="racquet_frame" />
-        <origin xyz="0.0 -0.125 0.0" rpy="0.0 0.78539816339 0.0" />
+        <origin xyz="0.0 0.0 0.125" rpy="-1.57079632679 0.0 0.0" />
       </joint>
       <joint name="plate_to_tool" type="fixed">

Commit message: Add kinova_bota_peg_plate_camera variant (hole plate with camera mount)
New EndEffector::PegPlateCamera on the Gen0 Bota sensor, exposed as robot
modules KinovaBotaPegPlateCamera / KinovaBotaPegPlateCameraCallib (urdf
kinova_bota_peg_plate_camera).

Same robot-side hole plate as peg_plate plus a camera mount rising in +z
(meshes/peg_plate_camera.STL, already in metres, same FT mounting rotation
rpy 0 -pi/2 -pi/2). Inertia computed from the mesh (uniform density) for the
measured mass of 0.695 kg of the modelled piece; the 70 g camera itself is
not modelled yet (add a camera frame/mass later). Bounding-box collision.

File: xacro/gen3_bota.in.xacro (robot description, xacro)
@@ -280,4 +280,37 @@
       <link name="tool"></link>
     </xacro:if>
+    <!-- Robot-side hole plate with a camera mount (Peg_in_Hole_plate_Camera_Robot_Handle.stl)
+         for collaborative peg-in-hole data collection. Same handle plate as 'peg_plate' plus a
+         camera mount rising in +z. Inertia computed from the mesh (uniform density) for the
+         measured mass of 0.695 kg of the modelled piece; the 70 g camera itself is NOT modelled
+         here (add it with a camera frame later). Inertia scales linearly with mass. -->
+    <xacro:if value="$(eval end_effector == 'peg_plate_camera')">
+      <link name="peg_plate_camera">
+        <inertial>
+          <origin xyz="0.14773 -0.00055 -0.01102" rpy="0 0 0" />
+          <mass value="0.695" />
+          <inertia ixx="5.539339E-03" ixy="-2.306877E-05" ixz="2.316990E-03"
+            iyy="1.262038E-02" iyz="8.946139E-05" izz="1.025269E-02" />
+        </inertial>
+        <visual name="peg_plate_camera">
+          <origin xyz="0.0 0.0 0.0" rpy="0 0 0" />
+          <geometry>
+            <!-- Mesh is already in metres, so no scaling. -->
+            <mesh filename="file://@CMAKE_SOURCE_DIR@/meshes/peg_plate_camera.STL" scale="1 1 1" />
+          </geometry>
+          <material name="">
+            <color rgba="0.2 0.4 0.8 1" />
+          </material>
+        </visual>
+        <!-- Bounding-box collision (398 x 180 x 290 mm) for cheap self-collision checks. -->
+        <collision>
+          <origin xyz="0.199 0.0 0.090" rpy="0 0 0" />
+          <geometry>
+            <box size="0.398 0.180 0.290" />
+          </geometry>
+        </collision>
+      </link>
+      <link name="tool"></link>
+    </xacro:if>
     <xacro:if value="$(eval bota_version == 'gena')">
       <joint name="kinova_to_FT" type="fixed">
@@ -382,4 +415,17 @@
       </joint>
     </xacro:if>
+    <xacro:if value="$(eval end_effector == 'peg_plate_camera')">
+      <!-- Same mounting as peg_plate: FT_x=plate_y, FT_y=plate_z, FT_z=plate_x (rpy 0 -pi/2 -pi/2). -->
+      <joint name="FT_to_peg_plate_camera" type="fixed">
+        <parent link="FT_sensor_tool_frame" />
+        <child link="peg_plate_camera" />
+        <origin xyz="0.0 0.0 0.0" rpy="0.0 -1.5707963267948966 -1.5707963267948966" />
+      </joint>
+      <joint name="peg_plate_camera_to_tool" type="fixed">
+        <parent link="peg_plate_camera" />
+        <child link="tool" />
+        <origin xyz="0.0 0.0 0.0" rpy="0.0 0.0 0.0" />
+      </joint>
+    </xacro:if>
   </xacro:if>
   <xacro:if value="$(eval gripper != '' and bota_version == 'gena')">

Commit message: fix: restore full calibration excitation range for plate/peg_plate variants
joint_4's calibration sweep was symmetrically shrunk (percentLimits) to avoid
a collision seen with the plate/peg_plate tools mounted, but the shrink also
threw away safe excitation range on the side that was never a problem,
starving the calibration solver's mass/CoM/offset identification of pose
diversity. Use explicit asymmetric lower/upper bounds instead: keep the
previously-tuned conservative side, restore the full range on the safe side.

Also fix plate's collision geometry in gen3_bota.in.xacro, which was a
leftover placeholder cylinder unrelated to the mesh's actual ~170x70x234mm
footprint, making any collision check against it meaningless.

File: xacro/gen3_bota.in.xacro (robot description, xacro)
@@ -176,8 +176,11 @@
           </material>
         </visual>
-        <collision>
-          <origin xyz="0 0 0.015" rpy="0 0 0" />
-          <geometry>
-            <cylinder radius="0.0075" length="0.03" />
+        <!-- Bounding-box collision (170 x 70 x 234 mm), computed from the plate.STL mesh
+             bounding box after applying the same visual origin rotation, since the mesh's
+             true footprint is much larger than a small placeholder shape. -->
+        <collision>
+          <origin xyz="0.0 0.0 0.102" rpy="0 0 0" />
+          <geometry>
+            <box size="0.170 0.070 0.234" />
           </geometry>
         </collision>

Commit message: feat(plate): Update plate end-effector to new CAD revision (226 g)
Replace plate.STL with the new printed revision and remodel the link from
the mesh. The new mesh is authored in metres (scale 1) in the plate link
frame rotated +90 deg about Z, so the visual origin carries that yaw.

Mass is 226 g (Bambu Studio estimate). Over the 183.2 cm^3 mesh volume that
is 1233 kg/m^3, essentially solid PLA, so the inertia is computed from the
mesh at uniform density.

The blade is now a 5 mm slab offset to one side of the wrist axis, spanning
y -0.035..-0.030, with the striking face on the plane y = -0.035.

Also fix two frame bugs the previous revision carried: the inertial origin
and the plate_to_racquet_frame joint were both written in mesh-frame
coordinates but interpreted in the link frame, which put racquet_frame off
the part entirely. Both are now expressed in the link frame, and the URDF
and the MuJoCo model agree on the plate and racquet frames.

File: xacro/gen3_bota.in.xacro (robot description, xacro)
@@ -161,26 +161,33 @@
     <xacro:if value="$(eval end_effector == 'plate')">
       <link name="plate">
-        <inertial>
-          <origin xyz="-1.58E-05 -9.40E-02 1.58E-05" rpy="0 0 0" />
-          <mass value="0.1" />
-          <inertia ixx="5.58925E-04" iyy="1.45301E-04" izz="5.58925E-04"
-                  ixy="1.52637E-07" ixz="6.50849E-05" iyz="-1.52637E-07" />
-        </inertial>
+        <!-- Measured mass 0.226 kg (Bambu Studio estimate for the printed part).
+             Over the 183.2 cm^3 mesh volume that is 1233 kg/m^3, i.e. essentially
+             solid PLA, so the inertia below is computed from the mesh at uniform
+             density. Expressed in the link frame, like the visual/collision below. -->
+        <inertial>
+          <origin xyz="1.81E-05 -2.51566E-02 9.55300E-02" rpy="0 0 0" />
+          <mass value="0.226" />
+          <inertia ixx="1.124629E-03" iyy="1.382903E-03" izz="3.658632E-04"
+                  ixy="-1.032380E-07" ixz="4.014063E-07" iyz="1.500394E-04" />
+        </inertial>
+        <!-- plate.STL is authored in metres, in the link frame rotated +90 deg about
+             Z, hence scale 1 and the yaw below. The blade is a 5 mm slab offset to
+             one side: its striking face is the plane y = -0.035 in the link frame. -->
         <visual name="plate">
-          <origin xyz="0.0 0.0 0.0" rpy="-1.57079632679 0 0.78539816339" />
-          <geometry>
-            <mesh filename="file://@CMAKE_SOURCE_DIR@/meshes/plate.STL" scale="0.001 0.001 0.001"/>
-          </geometry>
-          <material name="">
-            <color rgba="0.6902 0.61176 0.52941 1" />
-          </material>
-        </visual>
-        <!-- Bounding-box collision (170 x 70 x 234 mm), computed from the plate.STL mesh
-             bounding box after applying the same visual origin rotation, since the mesh's
-             true footprint is much larger than a small placeholder shape. -->
-        <collision>
-          <origin xyz="0.0 0.0 0.102" rpy="0 0 0" />
-          <geometry>
-            <box size="0.170 0.070 0.234" />
+          <origin xyz="0.0 0.0 0.0" rpy="0 0 -1.5707963267948966" />
+          <geometry>
+            <mesh filename="file://@CMAKE_SOURCE_DIR@/meshes/plate.STL" scale="1 1 1"/>
+          </geometry>
+          <material name="">
+            <color rgba="0.6902 0.61176 0.52941 1" />
+          </material>
+        </visual>
+        <!-- Bounding-box collision (170 x 70 x 233.4 mm) over the whole part, taken
+             from the plate.STL bounding box in the link frame. Only used for arm
+             self-collision pairs, so the hub envelope rather than the blade. -->
+        <collision>
+          <origin xyz="0.0 0.0 0.11172" rpy="0 0 0" />
+          <geometry>
+            <box size="0.170 0.070 0.2334" />
           </geometry>
         </collision>
@@ -323,8 +330,11 @@
       </joint>
       <link name="racquet_frame"></link>
+      <!-- Ball-balancing reference frame: origin on the blade mid-plane (the blade
+           spans y -0.035..-0.030 in the plate frame), +Z along the striking face
+           normal (-Y of the plate frame). -->
       <joint name="plate_to_racquet_frame" type="fixed">
         <parent link="plate" />
         <child link="racquet_frame" />
-        <origin xyz="0.0 -0.125 0.0" rpy="0.0 0.78539816339 0.0" />
+        <origin xyz="0.0 -0.0325 0.125" rpy="1.5707963267948966 0.0 0.0" />
       </joint>
       <joint name="plate_to_tool" type="fixed">

Commit message: fix(peg_plate_camera): model the camera and use the weighed plate mass
- peg_plate_camera 0.695 -> 0.700 kg (weighed), mesh inertia scaled to match
- new camera link on a fixed joint, 0.075 kg (weighed), at the top of the mount

The camera is not part of the printed mesh and was not modelled at all; the
xacro comment has flagged it as missing since the variant was added. Its
position comes from the couple channel of the 12-pose calibration run, the only
observable that can locate it -- the force channel sees the total mass and
nothing else. The fit places it at z = 0.2233 m in the plate link frame, at the
top of the camera mount and inside the existing collision box, which nothing in
the fit knew about.

Leaving it out put the tool CoM 2 cm off and doubled the generated calibration's
couple residual: 0.234 -> 0.093 N.m over 12 static poses.

Its own inertia is a placeholder. At 0.239 m from the plate CoM the
parallel-axis term is ~400x larger, so the shape given here does not matter.

File: xacro/gen3_bota.in.xacro (robot description, xacro)
@@ -282,14 +282,14 @@
     <!-- Robot-side hole plate with a camera mount (Peg_in_Hole_plate_Camera_Robot_Handle.stl)
          for collaborative peg-in-hole data collection. Same handle plate as 'peg_plate' plus a
-         camera mount rising in +z. Inertia computed from the mesh (uniform density) for the
-         measured mass of 0.695 kg of the modelled piece; the 70 g camera itself is NOT modelled
-         here (add it with a camera frame later). Inertia scales linearly with mass. -->
+         camera mount rising in +z. Inertia computed from the mesh (uniform density), scaled to
+         the weighed mass of 0.700 kg of the printed piece (was the 0.695 kg CAD estimate;
+         inertia scales linearly with mass). The camera itself is a separate link below. -->
     <xacro:if value="$(eval end_effector == 'peg_plate_camera')">
       <link name="peg_plate_camera">
         <inertial>
           <origin xyz="0.14773 -0.00055 -0.01102" rpy="0 0 0" />
-          <mass value="0.695" />
-          <inertia ixx="5.539339E-03" ixy="-2.306877E-05" ixz="2.316990E-03"
-            iyy="1.262038E-02" iyz="8.946139E-05" izz="1.025269E-02" />
+          <mass value="0.700" />
+          <inertia ixx="5.579190E-03" ixy="-2.323473E-05" ixz="2.333659E-03"
+            iyy="1.271117E-02" iyz="9.010500E-05" izz="1.032645E-02" />
         </inertial>
         <visual name="peg_plate_camera">
@@ -310,4 +310,21 @@
           </geometry>
         </collision>
+      </link>
+      <!-- The camera bolted to the top of the mount. It is not part of the printed mesh, so it
+           gets its own link. Mass 0.075 kg weighed on a scale; position derived from the couple
+           channel of the 12-pose calibration run (the force channel only sees the total mass, so
+           the couple is the only observable that locates it). It lands at the top of the camera
+           mount, inside the collision box above, which is an independent check on the fit.
+           Leaving it out biased the calibration by 75 g and, more importantly, put the tool CoM
+           2 cm off, which is why the camera variant's couple residual used to be 5x the plain
+           plate's. Its own inertia is a placeholder: at 0.239 m from the plate CoM the
+           parallel-axis term is 4.3e-3 kg.m^2, some 400x the camera's own, so the shape it is
+           given here does not matter. -->
+      <link name="camera">
+        <inertial>
+          <origin xyz="0.0 0.0 0.0" rpy="0 0 0" />
+          <mass value="0.075" />
+          <inertia ixx="1.0E-05" ixy="0.0" ixz="0.0" iyy="1.0E-05" iyz="0.0" izz="1.0E-05" />
+        </inertial>
       </link>
       <link name="tool"></link>
@@ -422,4 +439,9 @@
         <origin xyz="0.0 0.0 0.0" rpy="0.0 -1.5707963267948966 -1.5707963267948966" />
       </joint>
+      <joint name="peg_plate_camera_to_camera" type="fixed">
+        <parent link="peg_plate_camera" />
+        <child link="camera" />
+        <origin xyz="0.1882 -0.0270 0.2233" rpy="0.0 0.0 0.0" />
+      </joint>
       <joint name="peg_plate_camera_to_tool" type="fixed">
         <parent link="peg_plate_camera" />

Commit message: fix(racquet frame): restore the racquet_frame rotation sign
dd2af6d had already fixed this joint's rotation to rpy="-pi/2 0 0". 56be37f
("Fix raquet weight and Optional in CMakeLists") reverted the line wholesale back
to 4862da2's original xyz="0 -0.125 0" rpy="0 0.785 0", losing that fix silently --
devel-rl escaped it only because 5e5a850 reverted 56be37f there, which never
happened on this branch.

510c5eb then re-derived the origin for the new 226 g blade on top of the clobbered
line: the translation is right (xyz="0 -0.0325 0.125", blade mid-plane) but the
rotation carried the reverted +pi/2 forward. With +pi/2 the frame's +Z is -Y of the
plate frame, which at the q0 balancing stance points at the ground -- FK on the
matching MuJoCo model (ping_pong_kinova src/mjlab_kinova/robot/kinova.xml) puts
racquet_frame's +Z at world [0.0001, -0.0012, 1.0] only with -pi/2.

That mismatch is not cosmetic: the ball-balancing policy reads its end-effector
pose, velocity and the ball reset offset in this frame, so an inverted +Z means
training and deployment disagree by 180 degrees about X.

File: xacro/gen3_bota.in.xacro (robot description, xacro)
@@ -382,9 +382,11 @@
       <!-- Ball-balancing reference frame: origin on the blade mid-plane (the blade
            spans y -0.035..-0.030 in the plate frame), +Z along the striking face
-           normal (-Y of the plate frame). -->
+           normal (+Y of the plate frame, i.e. the y = -0.030 face). That is the face
+           pointing up at the q0 balancing stance; -Y points at the ground, and a ball
+           reset placed along it spawns underneath the blade. -->
       <joint name="plate_to_racquet_frame" type="fixed">
         <parent link="plate" />
         <child link="racquet_frame" />
-        <origin xyz="0.0 -0.0325 0.125" rpy="1.5707963267948966 0.0 0.0" />
+        <origin xyz="0.0 -0.0325 0.125" rpy="-1.5707963267948966 0.0 0.0" />
       </joint>
       <joint name="plate_to_tool" type="fixed">
