Commit message: Update calib variant logic and provide configuration for ForceSensorCalib controller

File: xacro/gen3.in.xacro (robot description, xacro)
@@ -25,5 +25,5 @@
   <xacro:arg name="simulation_controllers"
     default="$(find kortex_description)/arm/$(arg arm)/$(arg dof)dof/config/ros2_controllers.yaml" />
-  <xacro:arg name="DS4" default="false" />
+  <xacro:arg name="end_effector" default="none" />
   <xacro:arg name="bota" default="true" />
   <!-- import main macro -->
@@ -90,5 +90,5 @@
       </collision>
     </link>
-    <xacro:if value="$(arg DS4)">
+    <xacro:if value="$(eval end_effector == 'ds4')">
       <link name="DS4_adapter">
         <inertial>
@@ -149,5 +149,5 @@
       <origin xyz="0.0 0.0 0.0" rpy="0.0 0.0 0.0" />
     </joint>
-    <xacro:if value="$(arg DS4)">
+    <xacro:if value="$(eval end_effector == 'ds4')">
       <joint name="FT_to_DS4_adapter" type="fixed">
         <parent link="FT_sensor_wrench" />

File: xacro/gen3_bota.in.xacro (robot description, xacro)
@@ -25,6 +25,5 @@
   <xacro:arg name="simulation_controllers"
     default="$(find kortex_description)/arm/$(arg arm)/$(arg dof)dof/config/ros2_controllers.yaml" />
-  <xacro:arg name="DS4" default="false" />
-  <xacro:arg name="plate" default="false" />
+  <xacro:arg name="end_effector" default="none" />
   <xacro:arg name="bota" default="true" />
   <!-- import main macro -->
@@ -91,5 +90,8 @@
       </collision>
     </link>
-    <xacro:if value="$(arg DS4)">
+    <xacro:if value="$(eval end_effector == 'none')">
+      <link name="tool"></link>
+    </xacro:if>
+    <xacro:if value="$(eval end_effector == 'ds4')">
       <link name="DS4_adapter">
         <inertial>
@@ -138,7 +140,7 @@
         </collision>
       </link>
-      <link name="DS4_tool"></link>
-    </xacro:if>
-    <xacro:if value="$(arg plate)">
+      <link name="tool"></link>
+    </xacro:if>
+    <xacro:if value="$(eval end_effector == 'plate')">
       <link name="plate">
         <inertial>
@@ -148,8 +150,8 @@
             iyz="1.05961E-06" izz="8.81951E-05" />
         </inertial>
-        <visual name="ds4_adapter">
-          <origin xyz="0.0 0.0 0.0" rpy="0 0 0" />
-          <geometry>
-            <mesh filename="file://@CMAKE_SOURCE_DIR@/meshes/plate.STL" />
+        <visual name="plate">
+          <origin xyz="0.0 0.0 0.0" rpy="-1.57079632679 0 0.78539816339" />
+          <geometry>
+            <mesh filename="file://@CMAKE_SOURCE_DIR@/meshes/plate.STL" scale="0.001 0.001 0.001"/>
           </geometry>
           <material name="">
@@ -164,5 +166,31 @@
         </collision>
       </link>
-      <link name="plate_tool"></link>
+      <link name="tool"></link>
+    </xacro:if>
+    <xacro:if value="$(eval end_effector == 'screw')">
+      <link name="screw">
+        <inertial>
+          <origin xyz="-0.0001681638469675113 -0.0024779164507503317 0.059811455964133025" rpy="0 0 0" />
+          <mass value="0.0698" />
+          <inertia ixx="5.40350E-05" ixy="8.13203E-08" ixz="1.70226E-06" iyy="5.69809E-05"
+            iyz="1.05961E-06" izz="8.81951E-05" />
+        </inertial>
+        <visual name="screw">
+          <origin xyz="0.0 0.0 0.0" rpy="-1.57079632679 0 0" />
+          <geometry>
+            <mesh filename="file://@CMAKE_SOURCE_DIR@/meshes/screw.STL" scale="0.001 0.001 0.001" />
+          </geometry>
+          <material name="">
+            <color rgba="0.6902 0.61176 0.52941 1" />
+          </material>
+        </visual>
+        <collision>
+          <origin xyz="0 0 0.015" rpy="0 0 0" />
+          <geometry>
+            <cylinder radius="0.0075" length="0.03" />
+          </geometry>
+        </collision>
+      </link>
+      <link name="tool"></link>
     </xacro:if>
     <joint name="kinova_to_adapter" type="fixed">
@@ -176,5 +204,12 @@
       <origin xyz="0.0 0.0 0.0" rpy="0.0 0.0 0.0" />
     </joint>
-    <xacro:if value="$(arg DS4)">
+    <xacro:if value="$(eval end_effector == 'none')">
+      <joint name="FT_to_tool" type="fixed">
+        <parent link="FT_sensor_wrench" />
+        <child link="tool" />
+        <origin xyz="0.0 0.0 0.0" rpy="0.0 0.0 0.0" />
+      </joint>
+    </xacro:if>
+    <xacro:if value="$(eval end_effector == 'ds4')">
       <joint name="FT_to_DS4_adapter" type="fixed">
         <parent link="FT_sensor_wrench" />
@@ -189,9 +224,9 @@
       <joint name="DS4_to_tool" type="fixed">
         <parent link="DS4" />
-        <child link="DS4_tool" />
-        <origin xyz="0.0 0.0 0.0" rpy="0.0 0.0 0.0" />
-      </joint>
-    </xacro:if>
-    <xacro:if value="$(arg plate)">
+        <child link="tool" />
+        <origin xyz="0.0 0.0 0.0" rpy="0.0 0.0 0.0" />
+      </joint>
+    </xacro:if>
+    <xacro:if value="$(eval end_effector == 'plate')">
       <joint name="FT_to_plate" type="fixed">
         <parent link="FT_sensor_wrench" />
@@ -201,5 +236,17 @@
       <joint name="plate_to_tool" type="fixed">
         <parent link="plate" />
-        <child link="plate_tool" />
+        <child link="tool" />
+        <origin xyz="0.0 0.0 0.0" rpy="0.0 0.0 0.0" />
+      </joint>
+    </xacro:if>
+    <xacro:if value="$(eval end_effector == 'screw')">
+      <joint name="FT_to_screw" type="fixed">
+        <parent link="FT_sensor_wrench" />
+        <child link="screw" />
+        <origin xyz="0.0 0.0 0.0" rpy="0.0 0.0 0.0" />
+      </joint>
+      <joint name="screw_to_tool" type="fixed">
+        <parent link="screw" />
+        <child link="tool" />
         <origin xyz="0.0 0.0 0.0" rpy="0.0 0.0 0.0" />
       </joint>

Commit message: Add Kinova gripper variants and GenA Bota gripper support

File: xacro/gen3.in.xacro (robot description, xacro)
@@ -28,13 +28,18 @@
   <xacro:arg name="bota" default="true" />
   <xacro:arg name="bota_version" default="gen0" />
-  <!-- import main macro -->
-  <xacro:include filename="$(find kortex_description)/robots/kortex_robot.xacro" />
+  <!-- Load the arm directly so we can control what gets attached after the arm -->
+  <xacro:include filename="$(find kortex_description)/arms/gen3/7dof/urdf/gen3_macro.xacro" />
+  <xacro:if value="$(eval gripper == 'robotiq_2f_85')">
+    <xacro:include filename="$(find kortex_description)/grippers/robotiq_2f_85/urdf/robotiq_2f_85_macro.xacro" />
+  </xacro:if>
+  <xacro:if value="$(eval gripper == 'robotiq_2f_140')">
+    <xacro:include filename="$(find kortex_description)/grippers/robotiq_2f_140/urdf/robotiq_2f_140_macro.xacro" />
+  </xacro:if>
   <!-- convert to property to use substitution in function -->
   <xacro:property name="initial_positions_file" default="$(arg initial_positions_file)" />
   <!-- create link fixed to the "world" -->
   <link name="world" />
-  <xacro:load_robot
+  <xacro:load_arm
     parent="world"
-    arm="$(arg arm)"
     gripper="$(arg gripper)"
     gripper_joint_name="$(arg gripper_joint_name)"
@@ -57,5 +62,25 @@
     sim_isaac="$(arg sim_isaac)">
     <origin xyz="0 0 0" rpy="0 0 0" />
-  </xacro:load_robot>
+  </xacro:load_arm>
+  <xacro:if value="$(eval gripper == '')">
+    <link name="$(arg prefix)tool_frame"/>
+    <joint name="$(arg prefix)tool_frame_joint" type="fixed">
+      <origin xyz="0 0 0" rpy="0 0 0" />
+      <parent link="$(arg prefix)end_effector_link" />
+      <child link="$(arg prefix)tool_frame" />
+      <axis xyz="0 0 0" />
+    </joint>
+  </xacro:if>
+  <xacro:unless value="$(eval gripper == '')">
+    <xacro:load_gripper
+      parent="$(arg prefix)end_effector_link"
+      prefix="$(arg prefix)"
+      use_fake_hardware="$(arg use_fake_hardware)"
+      fake_sensor_commands="$(arg fake_sensor_commands)"
+      sim_gazebo="$(arg sim_gazebo)"
+      sim_isaac="$(arg sim_isaac)"
+      com_port="/dev/ttyUSB0"
+      use_internal_bus_gripper_comm="$(arg use_internal_bus_gripper_comm)" />
+  </xacro:unless>
   <xacro:if value="$(arg sim_gazebo)">
     <gazebo reference="world">

File: xacro/gen3_bota.in.xacro (robot description, xacro)
@@ -28,13 +28,18 @@
   <xacro:arg name="bota" default="true" />
   <xacro:arg name="bota_version" default="gen0" />
-  <!-- import main macro -->
-  <xacro:include filename="$(find kortex_description)/robots/kortex_robot.xacro" />
+  <!-- Load the arm directly so the tooling and the gripper can be attached explicitly -->
+  <xacro:include filename="$(find kortex_description)/arms/gen3/7dof/urdf/gen3_macro.xacro" />
+  <xacro:if value="$(eval gripper == 'robotiq_2f_85')">
+    <xacro:include filename="$(find kortex_description)/grippers/robotiq_2f_85/urdf/robotiq_2f_85_macro.xacro" />
+  </xacro:if>
+  <xacro:if value="$(eval gripper == 'robotiq_2f_140')">
+    <xacro:include filename="$(find kortex_description)/grippers/robotiq_2f_140/urdf/robotiq_2f_140_macro.xacro" />
+  </xacro:if>
   <!-- convert to property to use substitution in function -->
   <xacro:property name="initial_positions_file" default="$(arg initial_positions_file)" />
   <!-- create link fixed to the "world" -->
   <link name="world" />
-  <xacro:load_robot
+  <xacro:load_arm
     parent="world"
-    arm="$(arg arm)"
     gripper="$(arg gripper)"
     gripper_joint_name="$(arg gripper_joint_name)"
@@ -57,5 +62,5 @@
     sim_isaac="$(arg sim_isaac)">
     <origin xyz="0 0 0" rpy="0 0 0" />
-  </xacro:load_robot>
+  </xacro:load_arm>
   <xacro:if value="$(arg sim_gazebo)">
     <gazebo reference="world">
@@ -271,3 +276,14 @@
     </xacro:if>
   </xacro:if>
+  <xacro:if value="$(eval gripper != '' and bota_version == 'gena')">
+    <xacro:load_gripper
+      parent="tool"
+      prefix="$(arg prefix)"
+      use_fake_hardware="$(arg use_fake_hardware)"
+      fake_sensor_commands="$(arg fake_sensor_commands)"
+      sim_gazebo="$(arg sim_gazebo)"
+      sim_isaac="$(arg sim_isaac)"
+      com_port="/dev/ttyUSB0"
+      use_internal_bus_gripper_comm="$(arg use_internal_bus_gripper_comm)" />
+  </xacro:if>
   </robot>

Commit message: fix(rokubimini_description): stop using rokubimini_decription for compatibility with newer version of bota_driver

File: xacro/gen3.in.xacro (robot description, xacro)
@@ -87,5 +87,5 @@
     </xacro:if>
     <xacro:unless value="$(eval bota_version == 'gena')">
-      <xacro:include filename="$(find rokubimini_description)/urdf/BFT_SENS_ECAT_M8.urdf.xacro" />
+      <xacro:include filename="$(find bota_driver)/urdf/BFT_SENS_ECAT_M8.urdf.xacro" />
       <xacro:BFT_SENS_ECAT_M8 prefix="FT_sensor" />
     </xacro:unless>

File: xacro/gen3_bota.in.xacro (robot description, xacro)
@@ -73,5 +73,5 @@
     </xacro:if>
     <xacro:unless value="$(eval bota_version == 'gena')">
-      <xacro:include filename="$(find rokubimini_description)/urdf/BFT_SENS_ECAT_M8.urdf.xacro" />
+      <xacro:include filename="$(find bota_driver)/urdf/BFT_SENS_ECAT_M8.urdf.xacro" />
       <xacro:BFT_SENS_ECAT_M8 prefix="FT_sensor" />
       <link name="FT_sensor_tool_frame" />
@@ -211,4 +211,30 @@
       <link name="tool"></link>
     </xacro:if>
+    <xacro:if value="$(eval end_effector == 'hook')">
+      <link name="hook">
+        <inertial>
+          <origin xyz="4.40561E-05 1.22892E-02 -3.48748E-03" rpy="0 0 0" />
+          <mass value="0.0368" />
+          <inertia ixx="2.14342E-05" ixy="2.00498E-08" ixz="1.44079E-08" iyy="1.50275E-05"
+            iyz="-2.20625E-07" izz="3.50484E-05" />
+        </inertial>
+        <visual name="hook">
+          <origin xyz="0.0 0.0 0.0" rpy="0 0 0" />
+          <geometry>
+            <mesh filename="file://@CMAKE_SOURCE_DIR@/meshes/hook.STL" scale="0.001 0.001 0.001" />
+          </geometry>
+          <material name="">
+            <color rgba="0.6902 0.61176 0.52941 1" />
+          </material>
+        </visual>
+        <collision>
+          <origin xyz="0.0 0.0 0.0" rpy="0 0 0" />
+          <geometry>
+            <cylinder radius="0.0075" length="0.03" />
+          </geometry>
+        </collision>
+      </link>
+      <link name="tool"></link>
+    </xacro:if>
     <xacro:if value="$(eval bota_version == 'gena')">
       <joint name="kinova_to_FT" type="fixed">
@@ -278,4 +304,16 @@
       </joint>
     </xacro:if>
+    <xacro:if value="$(eval end_effector == 'hook')">
+      <joint name="FT_to_hook" type="fixed">
+        <parent link="FT_sensor_tool_frame" />
+        <child link="hook" />
+        <origin xyz="0.0 0.0 0.0" rpy="0.0 0.0 0.0" />
+      </joint>
+      <joint name="hook_to_tool" type="fixed">
+        <parent link="hook" />
+        <child link="tool" />
+        <origin xyz="0.0 0.0 0.0" rpy="0.0 0.0 0.0" />
+      </joint>
+    </xacro:if>
   </xacro:if>
   <xacro:if value="$(eval gripper != '' and bota_version == 'gena')">

Commit message: chore: delete unused stl

File: xacro/gen3.in.xacro (robot description, xacro)
@@ -26,5 +26,4 @@
     default="$(find kortex_description)/arm/$(arg arm)/$(arg dof)dof/config/ros2_controllers.yaml" />
   <xacro:arg name="end_effector" default="none" />
-  <xacro:arg name="bota" default="true" />
   <!-- import main macro -->
   <xacro:include filename="$(find kortex_description)/robots/kortex_robot.xacro" />
@@ -64,106 +63,3 @@
     </gazebo>
   </xacro:if>
-  <xacro:if value="$(arg bota)">
-    <xacro:include filename="$(find bota_driver)/urdf/BFT_SENS_ECAT_M8.urdf.xacro" />
-    <xacro:BFT_SENS_ECAT_M8 prefix="FT_sensor" />
-    <link name="FT_adapter">
-      <inertial>
-        <origin xyz="0.001329828523918 0.000509434161397 0.017297595549827" rpy="0 0 0" />
-        <mass value="0.12" />
-        <inertia ixx="5.40350E-05" ixy="8.13203E-08" ixz="1.70226E-06" iyy="5.69809E-05"
-          iyz="1.05961E-06" izz="8.81951E-05" />
-      </inertial>
-      <visual name="adapter">
-        <origin xyz="0 0 0.0" rpy="0 0 0" />
-        <geometry>
-          <mesh filename="file://@CMAKE_SOURCE_DIR@/meshes/adapter.STL" />
-        </geometry>
-        <material name="">
-          <color rgba="0.6902 0.61176 0.52941 1" />
-        </material>
-      </visual>
-      <collision>
-        <origin xyz="0 0 0.015" rpy="0 0 0" />
-        <geometry>
-          <cylinder radius="0.0075" length="0.03" />
-        </geometry>
-      </collision>
-    </link>
-    <xacro:if value="$(eval end_effector == 'ds4')">
-      <link name="DS4_adapter">
-        <inertial>
-          <origin xyz="-0.0001681638469675113 -0.0024779164507503317 0.059811455964133025" rpy="0 0 0" />
-          <mass value="0.0698" />
-          <inertia ixx="5.40350E-05" ixy="8.13203E-08" ixz="1.70226E-06" iyy="5.69809E-05"
-            iyz="1.05961E-06" izz="8.81951E-05" />
-        </inertial>
-        <visual name="ds4_adapter">
-          <origin xyz="0.0 0.0 0.0" rpy="0 0 0" />
-          <geometry>
-            <mesh filename="file://@CMAKE_SOURCE_DIR@/meshes/DS4_adapter.STL" />
-          </geometry>
-          <material name="">
-            <color rgba="0.6902 0.61176 0.52941 1" />
-          </material>
-        </visual>
-        <collision>
-          <origin xyz="0 0 0.015" rpy="0 0 0" />
-          <geometry>
-            <cylinder radius="0.0075" length="0.03" />
-          </geometry>
-        </collision>
-      </link>
-      <link name="DS4">
-        <inertial>
-          <origin xyz="0.0 0.0 0.045" rpy="0 0 0" />
-          <mass value="0.2162" />
-          <inertia ixx="5.40350E-05" ixy="8.13203E-08" ixz="1.70226E-06" iyy="5.69809E-05"
-            iyz="1.05961E-06" izz="8.81951E-05" />
-        </inertial>
-        <visual name="ds4">
-          <origin xyz="0.0 0.0 0.0" rpy="0 0 0" />
-          <geometry>
-            <box size="0.14 0.03 0.06" />
-          </geometry>
-          <material name="">
-            <color rgba="0.6902 0.61176 0.52941 1" />
-          </material>
-        </visual>
-        <collision>
-          <origin xyz="0 0 0.03" rpy="0 1.57 0" />
-          <geometry>
-            <cylinder radius="0.0075" length="0.14" />
-          </geometry>
-        </collision>
-      </link>
-      <link name="DS4_tool"></link>
-    </xacro:if>
-    <joint name="kinova_to_adapter" type="fixed">
-      <parent link="end_effector_link" />
-      <child link="FT_adapter" />
-      <origin xyz="0.0 0.0 0.03" rpy="0.0 0.0 0.0" />
-    </joint>
-    <joint name="adapter_to_FT" type="fixed">
-      <parent link="FT_adapter" />
-      <child link="FT_sensor_mounting" />
-      <origin xyz="0.0 0.0 0.0" rpy="0.0 0.0 0.0" />
-    </joint>
-    <xacro:if value="$(eval end_effector == 'ds4')">
-      <joint name="FT_to_DS4_adapter" type="fixed">
-        <parent link="FT_sensor_wrench" />
-        <child link="DS4_adapter" />
-        <origin xyz="0.0 0.0 0.0" rpy="0.0 0.0 0.0" />
-      </joint>
-      <joint name="DS4_adapter_to_DS4" type="fixed">
-        <parent link="DS4_adapter" />
-        <child link="DS4" />
-        <origin xyz="0.0 0.0 0.08" rpy="0.0 0.0 0.0" />
-      </joint>
-      <joint name="DS4_to_tool" type="fixed">
-        <parent link="DS4" />
-        <child link="DS4_tool" />
-        <origin xyz="0.0 0.0 0.0" rpy="0.0 0.0 0.0" />
-      </joint>
-    </xacro:if>
-  </xacro:if>
-  </robot>
+</robot>
