Commit message: fix: correct paths in xacro.in using CURRENT_SOURCE_DIR
These path would still be correct when mc_kinova is included as
submodule.

File: xacro/gen3.in.xacro (robot description, xacro)
@@ -77,5 +77,5 @@
         <origin xyz="0 0 0.0" rpy="0 0 0" />
         <geometry>
-          <mesh filename="file://@CMAKE_SOURCE_DIR@/meshes/adapter.STL" />
+          <mesh filename="file://@CMAKE_CURRENT_SOURCE_DIR@/meshes/adapter.STL" />
         </geometry>
         <material name="">
@@ -101,5 +101,5 @@
           <origin xyz="0.0 0.0 0.0" rpy="0 0 0" />
           <geometry>
-            <mesh filename="file://@CMAKE_SOURCE_DIR@/meshes/DS4_adapter.STL" />
+            <mesh filename="file://@CMAKE_CURRENT_SOURCE_DIR@/meshes/DS4_adapter.STL" />
           </geometry>
           <material name="">

File: xacro/gen3_bota.in.xacro (robot description, xacro)
@@ -77,5 +77,5 @@
         <origin xyz="0 0 0.0" rpy="0 0 0" />
         <geometry>
-          <mesh filename="file://@CMAKE_SOURCE_DIR@/meshes/adapter.STL" />
+          <mesh filename="file://@CMAKE_CURRENT_SOURCE_DIR@/meshes/adapter.STL" />
         </geometry>
         <material name="">
@@ -104,5 +104,5 @@
           <origin xyz="0.0 0.0 0.0" rpy="0 0 0" />
           <geometry>
-            <mesh filename="file://@CMAKE_SOURCE_DIR@/meshes/DS4_adapter.STL" />
+            <mesh filename="file://@CMAKE_CURRENT_SOURCE_DIR@/meshes/DS4_adapter.STL" />
           </geometry>
           <material name="">
@@ -153,5 +153,5 @@
           <origin xyz="0.0 0.0 0.0" rpy="-1.57079632679 0 0.78539816339" />
           <geometry>
-            <mesh filename="file://@CMAKE_SOURCE_DIR@/meshes/plate.STL" scale="0.001 0.001 0.001"/>
+            <mesh filename="file://@CMAKE_CURRENT_SOURCE_DIR@/meshes/plate.STL" scale="0.001 0.001 0.001"/>
           </geometry>
           <material name="">
@@ -179,5 +179,5 @@
           <origin xyz="0.0 0.0 0.0" rpy="-1.57079632679 0 0" />
           <geometry>
-            <mesh filename="file://@CMAKE_SOURCE_DIR@/meshes/screw.STL" scale="0.001 0.001 0.001" />
+            <mesh filename="file://@CMAKE_CURRENT_SOURCE_DIR@/meshes/screw.STL" scale="0.001 0.001 0.001" />
           </geometry>
           <material name="">
